File: hardware/drop-machine.sch (KiCad schematic (older format))
At the start: 22 parts

Commit message: Multiple wires for valve power connection
Parts:
- removed J?: Valves, symbol CONN_02X11
- added J?: CONN_02X10, symbol CONN_02X10
Connections:
- net +12V: now also J?.15 (P15), J?.16 (P16), J?.17 (P17), J?.18 (P18), J?.19 (P19), J?.20 (P20)
- net at Q?.3 (D): now also J?.1 (P1)
- net at Q?.3 (D): now also J?.3 (P3)
- net at Q?.3 (D): now also J?.5 (P5)
- net at Q?.3 (D): now also J?.7 (P7)
- net at Q?.3 (D): now also J?.9 (P9)
Changed lines of the file:
@@
 	1    0    0    -1
 $EndComp
-Wire Wire Line
-	1400 1500 1500 1500
-Wire Wire Line
-	5650 3400 5650 3050
-Wire Wire Line
-	2100 1800 2900 1800
-Connection ~ 2500 1800
-Wire Wire Line
-	4500 3100 4500 2700
-Wire Wire Line
-	4500 2700 4250 2700
-Wire Wire Line
-	2100 1500 1800 1500
-Wire Wire Line
-	5650 4000 6350 4000
-Wire Wire Line
-	5650 4100 6350 4100
-Wire Wire Line
-	6350 4200 6200 4200
-Wire Wire Line
-	6200 5600 3100 5600
-Wire Wire Line
-	3100 5600 3100 3400
-Wire Wire Line
-	3100 3400 3350 3400
 $Comp
 L +5V #PWR010
@@
 	1    0    0    -1
 $EndComp
-Wire Wire Line
-	7000 4200 6850 4200
-Wire Wire Line
-	6200 4200 6200 5600
-Wire Wire Line
-	5650 3900 6200 3900
-Wire Wire Line
-	6200 3900 6200 3700
-Wire Wire Line
-	6200 3700 7000 3700
-Wire Wire Line
-	7000 3700 7000 4100
-Wire Wire Line
-	7000 4100 6850 4100
 $Comp
 L Q_NMOS_SGD Q?
@@
 	1    7600 4700
 	1    0    0    -1
-$EndComp
-$Comp
-L CONN_02X11 J?
-U 1 1 5A817C2E
-P 8800 3750
-F 0 "J?" H 8800 4350 50  0000 C CNN
-F 1 "Valves" V 8800 3750 50  0000 C CNN
-F 2 "" H 8800 2550 50  0001 C CNN
-F 3 "" H 8800 2550 50  0001 C CNN
-	1    8800 3750
-	0    -1   -1   0
 $EndComp
 $Comp
@@
 	1    0    0    -1
 $EndComp
-Wire Wire Line
-	7700 4500 7700 4000
-Wire Wire Line
-	7700 4000 8300 4000
-Wire Wire Line
-	8400 4000 8400 4100
-Wire Wire Line
-	8400 4100 8250 4100
-Wire Wire Line
-	8250 4100 8250 4500
-Wire Wire Line
-	8800 4500 8800 4300
-Wire Wire Line
-	8800 4300 8500 4300
-Wire Wire Line
-	8500 4300 8500 4000
-Wire Wire Line
-	9350 4500 9350 4250
-Wire Wire Line
-	9350 4250 8600 4250
-Wire Wire Line
-	8600 4250 8600 4000
-Wire Wire Line
-	8700 4000 8700 4200
-Wire Wire Line
-	8700 4200 9900 4200
-Wire Wire Line
-	9900 4200 9900 4500
 $Comp
 L +12V #PWR017
@@
 	1    0    0    -1
 $EndComp
-Wire Wire Line
-	9300 4000 9500 4000
 Entry Wire Line
 	5800 4300 5900 4400
@@
 Entry Wire Line
 	9500 5300 9600 5200
-Wire Bus Line
-	9500 5300 5900 5300
-Wire Bus Line
-	5900 5300 5900 4400
-Wire Wire Line
-	9600 5000 9600 5200
-Wire Wire Line
-	9050 5000 9050 5200
-Wire Wire Line
-	8500 5000 8500 5200
-Wire Wire Line
-	7950 5000 7950 5200
-Wire Wire Line
-	7400 5000 7400 5200
-Wire Wire Line
-	5800 4300 5650 4300
-Wire Wire Line
-	5800 4400 5650 4400
-Wire Wire Line
-	5800 4500 5650 4500
-Wire Wire Line
-	5800 4600 5650 4600
-Wire Wire Line
-	5800 4700 5650 4700
 NoConn ~ 5650 3500
 NoConn ~ 5650 3600
@@
 NoConn ~ 3350 3700
 NoConn ~ 3350 3900
+$Comp
+L CONN_02X10 J?
+U 1 1 5A81D8F6
+P 8750 3750
+F 0 "J?" H 8750 4300 50  0000 C CNN
+F 1 "CONN_02X10" V 8750 3750 50  0000 C CNN
+F 2 "" H 8750 2550 50  0001 C CNN
+F 3 "" H 8750 2550 50  0001 C CNN
+	1    8750 3750
+	0    -1   -1   0
+$EndComp
+Wire Wire Line
+	1400 1500 1500 1500
+Wire Wire Line
+	5650 3400 5650 3050
+Wire Wire Line
+	2100 1800 2900 1800
+Connection ~ 2500 1800
+Wire Wire Line
+	4500 3100 4500 2700
+Wire Wire Line
+	4500 2700 4250 2700
+Wire Wire Line
+	2100 1500 1800 1500
+Wire Wire Line
+	5650 4000 6350 4000
+Wire Wire Line
+	5650 4100 6350 4100
+Wire Wire Line
+	6350 4200 6200 4200
+Wire Wire Line
+	6200 5600 3100 5600
+Wire Wire Line
+	3100 5600 3100 3400
+Wire Wire Line
+	3100 3400 3350 3400
+Wire Wire Line
+	7000 4200 6850 4200
+Wire Wire Line
+	6200 4200 6200 5600
+Wire Wire Line
+	5650 3900 6200 3900
+Wire Wire Line
+	6200 3900 6200 3700
+Wire Wire Line
+	6200 3700 7000 3700
+Wire Wire Line
+	7000 3700 7000 4100
+Wire Wire Line
+	7000 4100 6850 4100
+Wire Wire Line
+	7700 4500 7700 4000
+Wire Wire Line
+	7700 4000 8300 4000
+Wire Wire Line
+	8400 4000 8400 4100
+Wire Wire Line
+	8400 4100 8250 4100
+Wire Wire Line
+	8250 4100 8250 4500
+Wire Wire Line
+	8800 4500 8800 4300
+Wire Wire Line
+	8800 4300 8500 4300
+Wire Wire Line
+	8500 4300 8500 4000
+Wire Wire Line
+	9350 4500 9350 4250
+Wire Wire Line
+	9350 4250 8600 4250
+Wire Wire Line
+	8600 4250 8600 4000
+Wire Wire Line
+	8700 4000 8700 4200
+Wire Wire Line
+	8700 4200 9900 4200
+Wire Wire Line
+	9900 4200 9900 4500
+Wire Bus Line
+	5900 5300 9500 5300
+Wire Bus Line
+	5900 4400 5900 5300
+Wire Wire Line
+	9600 5000 9600 5200
+Wire Wire Line
+	9050 5000 9050 5200
+Wire Wire Line
+	8500 5000 8500 5200
+Wire Wire Line
+	7950 5000 7950 5200
+Wire Wire Line
+	7400 5000 7400 5200
+Wire Wire Line
+	5800 4300 5650 4300
+Wire Wire Line
+	5800 4400 5650 4400
+Wire Wire Line
+	5800 4500 5650 4500
+Wire Wire Line
+	5800 4600 5650 4600
+Wire Wire Line
+	5800 4700 5650 4700
+Connection ~ 9200 4000
+Connection ~ 9100 4000
+Wire Wire Line
+	9000 4000 9500 4000
+Wire Wire Line
+	9300 3500 9300 4000
+Wire Wire Line
+	9000 3500 9300 3500
+Connection ~ 9300 4000
+Connection ~ 9200 3500
+Connection ~ 9100 3500
 $EndSCHEMATC
